File: Door_Controller/CAN.sch (KiCad schematic (older format))
At the start: 13 parts

Commit message: rm CAN continuity
Parts:
- removed C? (x2): C, symbol Device:C
- removed Q?: 2N2219, Package_TO_SOT_THT:TO-39-3, symbol Transistor_BJT:2N2219
- removed R? (x5): R_US, symbol Device:R_US
Connections:
- net labels removed: CAN_IN_CONTA, CAN_IN_CONTB, CAN_IN_CONT_SNS, CAN_OUT_CONTA, CAN_OUT_CONTB, CAN_OUT_CONT_SNS
- wire segments 47 -> 22
Changed lines of the file:
@@
 	1    0    0    -1
 $EndComp
-Text HLabel 1350 1750 0    50   Input ~ 0
-CAN_IN_CONTA
-Text HLabel 1350 2000 0    50   Output ~ 0
-CAN_IN_CONTB
-Text HLabel 1300 4100 0    50   Input ~ 0
-CAN_OUT_CONTB
-Text HLabel 1300 3750 0    50   Output ~ 0
-CAN_OUT_CONTA
-$Comp
-L power:+BATT #PWR?
-U 1 1 5FB18612
-P 1800 3750
-F 0 "#PWR?" H 1800 3600 50  0001 C CNN
-F 1 "+BATT" H 1815 3923 50  0000 C CNN
-F 2 "" H 1800 3750 50  0001 C CNN
-F 3 "" H 1800 3750 50  0001 C CNN
-	1    1800 3750
-	1    0    0    -1
-$EndComp
-Wire Wire Line
-	1800 3750 1300 3750
-$Comp
-L Device:R_US R?
-U 1 1 5FB18D69
-P 1800 4400
-F 0 "R?" H 1868 4446 50  0000 L CNN
-F 1 "R_US" H 1868 4355 50  0000 L CNN
-F 2 "" V 1840 4390 50  0001 C CNN
-F 3 "~" H 1800 4400 50  0001 C CNN
-	1    1800 4400
-	1    0    0    -1
-$EndComp
-$Comp
-L Device:R_US R?
-U 1 1 5FB195F6
-P 1800 5000
-F 0 "R?" H 1868 5046 50  0000 L CNN
-F 1 "R_US" H 1868 4955 50  0000 L CNN
-F 2 "" V 1840 4990 50  0001 C CNN
-F 3 "~" H 1800 5000 50  0001 C CNN
-	1    1800 5000
-	1    0    0    -1
-$EndComp
-Wire Wire Line
-	1800 5300 1800 5250
-Wire Wire Line
-	1800 4850 1800 4750
-Wire Wire Line
-	1800 4250 1800 4100
-Wire Wire Line
-	1800 4100 1300 4100
-$Comp
-L Device:R_US R?
-U 1 1 5FB1F68F
-P 1750 2300
-F 0 "R?" H 1818 2346 50  0000 L CNN
-F 1 "R_US" H 1818 2255 50  0000 L CNN
-F 2 "" V 1790 2290 50  0001 C CNN
-F 3 "~" H 1750 2300 50  0001 C CNN
-	1    1750 2300
-	1    0    0    -1
-$EndComp
-$Comp
-L Device:R_US R?
-U 1 1 5FB20876
-P 1750 2850
-F 0 "R?" H 1818 2896 50  0000 L CNN
-F 1 "R_US" H 1818 2805 50  0000 L CNN
-F 2 "" V 1790 2840 50  0001 C CNN
-F 3 "~" H 1750 2850 50  0001 C CNN
-	1    1750 2850
-	1    0    0    -1
-$EndComp
-Wire Wire Line
-	1350 1750 1750 1750
-Wire Wire Line
-	1750 1750 1750 2000
-Wire Wire Line
-	1350 2000 1750 2000
-Connection ~ 1750 2000
-Wire Wire Line
-	1750 2000 1750 2150
-Wire Wire Line
-	1750 2450 1750 2550
-Wire Wire Line
-	1750 3000 1750 3100
-Text HLabel 2550 2550 2    50   Output ~ 0
-CAN_IN_CONT_SNS
-Text HLabel 2550 4750 2    50   Output ~ 0
-CAN_OUT_CONT_SNS
-Wire Wire Line
-	2550 2550 1750 2550
-Connection ~ 1750 2550
-Wire Wire Line
-	1750 2550 1750 2700
-Wire Wire Line
-	2550 4750 1800 4750
-Connection ~ 1800 4750
-Wire Wire Line
-	1800 4750 1800 4550
-$Comp
-L Device:C C?
-U 1 1 5FB22722
-P 1500 5000
-F 0 "C?" H 1615 5046 50  0000 L CNN
-F 1 "C" H 1615 4955 50  0000 L CNN
-F 2 "" H 1538 4850 50  0001 C CNN
-F 3 "~" H 1500 5000 50  0001 C CNN
-	1    1500 5000
-	1    0    0    -1
-$EndComp
-$Comp
-L Device:C C?
-U 1 1 5FB2321D
-P 1450 2850
-F 0 "C?" H 1565 2896 50  0000 L CNN
-F 1 "C" H 1565 2805 50  0000 L CNN
-F 2 "" H 1488 2700 50  0001 C CNN
-F 3 "~" H 1450 2850 50  0001 C CNN
-	1    1450 2850
-	1    0    0    -1
-$EndComp
-Wire Wire Line
-	1450 2700 1450 2550
-Wire Wire Line
-	1450 2550 1750 2550
-Wire Wire Line
-	1450 3000 1450 3100
-Wire Wire Line
-	1450 3100 1750 3100
-Connection ~ 1750 3100
-Wire Wire Line
-	1750 3100 1750 3200
-Wire Wire Line
-	1500 4850 1500 4750
-Wire Wire Line
-	1500 4750 1800 4750
-Wire Wire Line
-	1500 5150 1500 5250
-Wire Wire Line
-	1500 5250 1800 5250
-Connection ~ 1800 5250
-Wire Wire Line
-	1800 5250 1800 5150
 Text HLabel 4550 3000 0    50   BiDi ~ 0
 CANH_IN
@@
 	7050 4650 4650 4650
 $Comp
-L Transistor_BJT:2N2219 Q?
-U 1 1 5FB39FFD
-P 5350 4950
-F 0 "Q?" H 5540 4996 50  0000 L CNN
-F 1 "2N2219" H 5540 4905 50  0000 L CNN
-F 2 "Package_TO_SOT_THT:TO-39-3" H 5550 4875 50  0001 L CIN
-F 3 "http://www.onsemi.com/pub_link/Collateral/2N2219-D.PDF" H 5350 4950 50  0001 L CNN
-	1    5350 4950
-	1    0    0    -1
-$EndComp
-$Comp
-L Device:R_US R?
-U 1 1 5FB3BEA1
-P 5450 5450
-F 0 "R?" H 5518 5496 50  0000 L CNN
-F 1 "R_US" H 5518 5405 50  0000 L CNN
-F 2 "" V 5490 5440 50  0001 C CNN
-F 3 "~" H 5450 5450 50  0001 C CNN
-	1    5450 5450
-	1    0    0    -1
-$EndComp
-$Comp
 L power:Earth #PWR?
 U 1 1 5FB4209F
@@
 	1    0    0    -1
 $EndComp
-$Comp
-L power:Earth #PWR?
-U 1 1 5FB4461B
-P 1800 5300
-F 0 "#PWR?" H 1800 5050 50  0001 C CNN
-F 1 "Earth" H 1800 5150 50  0001 C CNN
-F 2 "" H 1800 5300 50  0001 C CNN
-F 3 "~" H 1800 5300 50  0001 C CNN
-	1    1800 5300
-	1    0    0    -1
-$EndComp
-$Comp
-L power:Earth #PWR?
-U 1 1 5FB44FD5
-P 1750 3200
-F 0 "#PWR?" H 1750 2950 50  0001 C CNN
-F 1 "Earth" H 1750 3050 50  0001 C CNN
-F 2 "" H 1750 3200 50  0001 C CNN
-F 3 "~" H 1750 3200 50  0001 C CNN
-	1    1750 3200
-	1    0    0    -1
-$EndComp
-$Comp
-L power:Earth #PWR?
-U 1 1 5FB4595E
-P 7100 5350
-F 0 "#PWR?" H 7100 5100 50  0001 C CNN
-F 1 "Earth" H 7100 5200 50  0001 C CNN
-F 2 "" H 7100 5350 50  0001 C CNN
-F 3 "~" H 7100 5350 50  0001 C CNN
-	1    7100 5350
-	0    -1   -1   0
-$EndComp
 $EndSCHEMATC
