File: Door_Controller/Micro.sch (KiCad schematic (older format))
At the start: 7 parts, among them U1 PIC18F26K83-E_SP

Commit message: convert grounds to earths
Connections:
- net labels added: Earth
- net labels removed: GNDD
Changed lines of the file:
@@
-$EndComp
-$Comp
-L power:GNDD #PWR?
-U 1 1 5FAB9EE1
-P 1450 2250
-F 0 "#PWR?" H 1450 2000 50  0001 C CNN
-F 1 "GNDD" H 1454 2095 50  0000 C CNN
-F 2 "" H 1450 2250 50  0001 C CNN
-F 3 "" H 1450 2250 50  0001 C CNN
-	1    1450 2250
-	1    0    0    -1
 $EndComp
 $Comp
@@
 Wire Wire Line
 	2650 1750 2850 1750
-$Comp
-L power:GNDD #PWR?
-U 1 1 5FAD196A
-P 2650 2300
-F 0 "#PWR?" H 2650 2050 50  0001 C CNN
-F 1 "GNDD" H 2654 2145 50  0000 C CNN
-F 2 "" H 2650 2300 50  0001 C CNN
-F 3 "" H 2650 2300 50  0001 C CNN
-	1    2650 2300
-	1    0    0    -1
-$EndComp
 Wire Wire Line
 	2650 2300 2650 1850
@@
 Wire Wire Line
 	7500 5200 8150 5200
+$Comp
+L power:Earth #PWR?
+U 1 1 5FB40AA5
+P 1450 2250
+F 0 "#PWR?" H 1450 2000 50  0001 C CNN
+F 1 "Earth" H 1450 2100 50  0001 C CNN
+F 2 "" H 1450 2250 50  0001 C CNN
+F 3 "~" H 1450 2250 50  0001 C CNN
+	1    1450 2250
+	1    0    0    -1
+$EndComp
+$Comp
+L power:Earth #PWR?
+U 1 1 5FB4135C
+P 2650 2300
+F 0 "#PWR?" H 2650 2050 50  0001 C CNN
+F 1 "Earth" H 2650 2150 50  0001 C CNN
+F 2 "" H 2650 2300 50  0001 C CNN
+F 3 "~" H 2650 2300 50  0001 C CNN
+	1    2650 2300
+	1    0    0    -1
+$EndComp
 $EndSCHEMATC
