File: Door_Controller/Motor_Controller_Pole.sch (KiCad schematic (older format))
At the start: 8 parts

Commit message: WIP motor poles
Other:
- note added: "Low Current MOSFET"
Changed lines of the file:
@@
 $Descr A4 11693 8268
 encoding utf-8
-Sheet 6 7
+Sheet 8 8
 Title ""
 Date ""
@@
 AR Path="/5FB4C28C/606144ED/6065772F" Ref="Q?"  Part="2"
 AR Path="/5FB4C28C/60652F73/6065772F" Ref="Q?"  Part="2"
+AR Path="/5FB4C28C/60688E8B/6065772F" Ref="Q?"  Part="2"
 F 0 "Q?" H 5094 2600 50  0000 L CNN
 F 1 "TSM8568CS_B1611" H 5496 2664 50  0001 C CNN
@@
 AR Path="/5FB4C28C/606144ED/6065773C" Ref="Q?"  Part="1"
 AR Path="/5FB4C28C/60652F73/6065773C" Ref="Q?"  Part="1"
+AR Path="/5FB4C28C/60688E8B/6065773C" Ref="Q?"  Part="1"
 F 0 "Q?" H 5094 4000 50  0000 L CNN
 F 1 "TSM8568CS_B1611" H 5496 4064 50  0001 C CNN
@@
 AR Path="/5FB4C28C/606144ED/60657745" Ref="R?"  Part="1"
 AR Path="/5FB4C28C/60652F73/60657745" Ref="R?"  Part="1"
+AR Path="/5FB4C28C/60688E8B/60657745" Ref="R?"  Part="1"
 F 0 "R?" V 4450 2600 50  0000 C CNN
 F 1 "R" V 4350 2600 50  0000 C CNN
@@
 AR Path="/5FB4C28C/606144ED/60657752" Ref="R?"  Part="1"
 AR Path="/5FB4C28C/60652F73/60657752" Ref="R?"  Part="1"
+AR Path="/5FB4C28C/60688E8B/60657752" Ref="R?"  Part="1"
 F 0 "R?" V 4700 3000 50  0000 L CNN
 F 1 "R" V 4600 3000 50  0000 L CNN
@@
 AR Path="/5FB4C28C/606144ED/60657763" Ref="R?"  Part="1"
 AR Path="/5FB4C28C/60652F73/60657763" Ref="R?"  Part="1"
+AR Path="/5FB4C28C/60688E8B/60657763" Ref="R?"  Part="1"
 F 0 "R?" V 6600 3750 50  0000 C CNN
 F 1 "100" V 6500 3750 50  0000 C CNN
@@
 U 1 1 60658886
 P 4950 4450
+AR Path="/5FB4C28C/60652F73/60658886" Ref="#PWR?"  Part="1"
+AR Path="/5FB4C28C/60688E8B/60658886" Ref="#PWR?"  Part="1"
 F 0 "#PWR?" H 4950 4200 50  0001 C CNN
 F 1 "Earth" H 4950 4300 50  0001 C CNN
@@
 U 1 1 6065D388
 P 2900 3550
+AR Path="/5FB4C28C/60652F73/6065D388" Ref="#PWR?"  Part="1"
+AR Path="/5FB4C28C/60688E8B/6065D388" Ref="#PWR?"  Part="1"
 F 0 "#PWR?" H 2900 3300 50  0001 C CNN
 F 1 "Earth" H 2900 3400 50  0001 C CNN
@@
 U 1 1 6065FAA7
 P 7800 3750
+AR Path="/5FB4C28C/60652F73/6065FAA7" Ref="U?"  Part="1"
+AR Path="/5FB4C28C/60688E8B/6065FAA7" Ref="U?"  Part="1"
 F 0 "U?" H 7850 4536 60  0000 C CNN
 F 1 "SN74LV1T04DCKR" H 7850 4430 60  0000 C CNN
@@
 U 1 1 60661651
 P 6850 3350
+AR Path="/5FB4C28C/60652F73/60661651" Ref="#PWR?"  Part="1"
+AR Path="/5FB4C28C/60688E8B/60661651" Ref="#PWR?"  Part="1"
 F 0 "#PWR?" H 6850 3200 50  0001 C CNN
 F 1 "+5V" H 6865 3523 50  0000 C CNN
@@
 U 1 1 60662854
 P 8800 4350
+AR Path="/5FB4C28C/60652F73/60662854" Ref="#PWR?"  Part="1"
+AR Path="/5FB4C28C/60688E8B/60662854" Ref="#PWR?"  Part="1"
 F 0 "#PWR?" H 8800 4100 50  0001 C CNN
 F 1 "Earth" H 8800 4200 50  0001 C CNN
@@
 AR Path="/5FB4C28C/606144ED/60666436" Ref="R?"  Part="1"
 AR Path="/5FB4C28C/60652F73/60666436" Ref="R?"  Part="1"
+AR Path="/5FB4C28C/60688E8B/60666436" Ref="R?"  Part="1"
 F 0 "R?" V 9050 3750 50  0000 C CNN
 F 1 "100" V 8950 3750 50  0000 C CNN
@@
 U 1 1 60675630
 P 3400 3250
+AR Path="/5FB4C28C/60652F73/60675630" Ref="Q?"  Part="1"
+AR Path="/5FB4C28C/60688E8B/60675630" Ref="Q?"  Part="1"
 F 0 "Q?" V 3875 3350 50  0000 C CNN
 F 1 "2N7002,215" V 3966 3350 50  0000 C CNN
@@
 Wire Wire Line
 	3400 3250 3400 3050
+Text Notes 4050 3300 2    39   ~ 0
+Low Current MOSFET
 $EndSCHEMATC
